Commit message: arm default inertias

File: urdf/andrzej_arms.xacro (robot description, xacro)
@@ -28,4 +28,5 @@
         <xacro:call macro="arm_${arm_name}_link_${link_name}_visual"/>
       </visual>
+      <xacro:call macro="arm_${arm_name}_link_${link_name}_inertia"/>
     </link>
     <joint name="arm_${arm_name}_joint_${link_name}" type="revolute">

File: urdf/andrzej_arms_spec.xacro (robot description, xacro)
@@ -124,3 +124,63 @@
     <origin xyz="0 0 .05"/>
   </xacro:macro>
+  <xacro:macro name="arm_1_link_1_inertia">
+    <inertial>
+      <mass value="0.1" />
+      <inertia ixx="1.0" ixy="0.0" ixz="0.0" iyy="1.0" iyz="0.0" izz="1.0" />
+    </inertial>
+  </xacro:macro>
+  <xacro:macro name="arm_1_link_2_inertia">
+    <inertial>
+      <mass value="0.1" />
+      <inertia ixx="1.0" ixy="0.0" ixz="0.0" iyy="1.0" iyz="0.0" izz="1.0" />
+    </inertial>
+  </xacro:macro>
+  <xacro:macro name="arm_1_link_3_inertia">
+    <inertial>
+      <mass value="0.1" />
+      <inertia ixx="1.0" ixy="0.0" ixz="0.0" iyy="1.0" iyz="0.0" izz="1.0" />
+    </inertial>
+  </xacro:macro>
+  <xacro:macro name="arm_1_link_4_inertia">
+    <inertial>
+      <mass value="0.1" />
+      <inertia ixx="1.0" ixy="0.0" ixz="0.0" iyy="1.0" iyz="0.0" izz="1.0" />
+    </inertial>
+  </xacro:macro>
+  <xacro:macro name="arm_1_link_5_inertia">
+    <inertial>
+      <mass value="0.1" />
+      <inertia ixx="1.0" ixy="0.0" ixz="0.0" iyy="1.0" iyz="0.0" izz="1.0" />
+    </inertial>
+  </xacro:macro>
+  <xacro:macro name="arm_2_link_1_inertia">
+    <inertial>
+      <mass value="0.1" />
+      <inertia ixx="1.0" ixy="0.0" ixz="0.0" iyy="1.0" iyz="0.0" izz="1.0" />
+    </inertial>
+  </xacro:macro>
+  <xacro:macro name="arm_2_link_2_inertia">
+    <inertial>
+      <mass value="0.1" />
+      <inertia ixx="1.0" ixy="0.0" ixz="0.0" iyy="1.0" iyz="0.0" izz="1.0" />
+    </inertial>
+  </xacro:macro>
+  <xacro:macro name="arm_2_link_3_inertia">
+    <inertial>
+      <mass value="0.1" />
+      <inertia ixx="1.0" ixy="0.0" ixz="0.0" iyy="1.0" iyz="0.0" izz="1.0" />
+    </inertial>
+  </xacro:macro>
+  <xacro:macro name="arm_2_link_4_inertia">
+    <inertial>
+      <mass value="0.1" />
+      <inertia ixx="1.0" ixy="0.0" ixz="0.0" iyy="1.0" iyz="0.0" izz="1.0" />
+    </inertial>
+  </xacro:macro>
+  <xacro:macro name="arm_2_link_5_inertia">
+    <inertial>
+      <mass value="0.1" />
+      <inertia ixx="1.0" ixy="0.0" ixz="0.0" iyy="1.0" iyz="0.0" izz="1.0" />
+    </inertial>
+  </xacro:macro>
 </robot>
