Commit message: mass as param

File: urdf/andrzej.xacro (robot description, xacro)
@@ -1,4 +1,5 @@
 <?xml version="1.0"?>
 <robot name="andrzej" xmlns:xacro="http://ros.org/wiki/xacro">
+  <!-- Dimensions -->
   <xacro:property name="base_width" value=".4" />
   <xacro:property name="base_length" value=".6" />
@@ -6,4 +7,8 @@
   <xacro:property name="wheel_diam" value=".1" />
   <xacro:property name="wheel_width" value=".04" />
+  <!-- Masses-->
+  <xacro:property name="base_mass" value="5" />
+  <xacro:property name="wheel_mass" value="0.3" />
+  <!-- Constants -->
   <xacro:property name="pi" value="3.1415926535897931" />
   <xacro:include filename="$(find andrzej_description)/urdf/materials.xacro" />

File: urdf/andrzej_base.xacro (robot description, xacro)
@@ -13,5 +13,5 @@
       </geometry>
     </collision>
-    <xacro:default_inertial mass="10"/>
+    <xacro:default_inertial mass="${base_mass}"/>
   </link>
   <xacro:macro name="wheel" params="prefix reflect_x reflect_y">
@@ -30,5 +30,5 @@
         </geometry>
       </collision>
-      <xacro:default_inertial mass="1"/>
+      <xacro:default_inertial mass="${wheel_mass}"/>
     </link>
     <joint name="${prefix}_wheel_joint" type="continuous">

Commit message: using inorder xacro, added visual arms, no grippers

File: urdf/andrzej.xacro (robot description, xacro)
@@ -10,6 +10,5 @@
   <xacro:property name="base_mass" value="5" />
   <xacro:property name="wheel_mass" value="0.3" />
-  <!-- Constants -->
-  <xacro:property name="pi" value="3.1415926535897931" />
+  <xacro:property name="arm_base_mass" value="0.2" />
   <xacro:include filename="$(find andrzej_description)/urdf/materials.xacro" />
   <xacro:macro name="default_inertial" params="mass">

File: urdf/andrzej_arms.xacro (robot description, xacro)
@@ -1,3 +1,48 @@
 <?xml version="1.0"?>
 <robot name="andrzej" xmlns:xacro="http://ros.org/wiki/xacro">
+  <xacro:include filename="$(find andrzej_description)/urdf/andrzej_arms_spec.xacro" />
+  <xacro:macro name="arm_base" params="arm_name reflect">
+    <link name="arm_${arm_name}_link_0">
+      <visual>
+        <geometry>
+          <box size="${arm_base_length} ${arm_base_width} ${arm_base_height}"/>
+        </geometry>
+        <material name="orange"/>
+      </visual>
+      <collision>
+        <geometry>
+          <box size="${arm_base_length} ${arm_base_width} ${arm_base_height}"/>
+        </geometry>
+      </collision>
+      <xacro:default_inertial mass="${arm_base_mass}"/>
+    </link>
+    <joint name="platform_to_arm_${arm_name}" type="fixed">
+      <parent link="base_link"/>
+      <child link="arm_${arm_name}_link_0"/>
+      <origin xyz="${base_length*reflect/4} 0 ${(base_height+arm_base_height)/2}"/>
+    </joint>
+  </xacro:macro>
+  <xacro:macro name="arm_link" params="arm_name link_name">
+    <link name="arm_${arm_name}_link_${link_name}">
+      <visual>
+        <xacro:call macro="arm_${arm_name}_link_${link_name}_visual"/>
+      </visual>
+    </link>
+    <joint name="arm_${arm_name}_joint_${link_name}" type="revolute">
+      <xacro:call macro="arm_${arm_name}_joint_${link_name}_spec"/>
+      <parent link="arm_${arm_name}_link_${link_name-1}"/>
+      <child link="arm_${arm_name}_link_${link_name}"/>
+    </joint>
+  </xacro:macro>
+  <xacro:macro name="arm" params="arm_name">
+    <xacro:arm_link arm_name="${arm_name}" link_name="1"/>
+    <xacro:arm_link arm_name="${arm_name}" link_name="2"/>
+    <xacro:arm_link arm_name="${arm_name}" link_name="3"/>
+    <xacro:arm_link arm_name="${arm_name}" link_name="4"/>
+    <xacro:arm_link arm_name="${arm_name}" link_name="5"/>
+  </xacro:macro>
+  <xacro:call macro="arm_base" arm_name="1" reflect="1" />
+  <xacro:call macro="arm_base" arm_name="2" reflect="-1" />
+  <xacro:call macro="arm" arm_name="1"/>
+  <xacro:call macro="arm" arm_name="2"/>
 </robot>

Commit message: gazebo ros control drop 1, added inertia-less base-footprint

File: urdf/andrzej.xacro (robot description, xacro)
@@ -18,4 +18,5 @@
     </inertial>
   </xacro:macro>
+  <xacro:include filename="$(find andrzej_description)/urdf/andrzej.gazebo" />
   <xacro:include filename="$(find andrzej_description)/urdf/andrzej_base.xacro" />
   <xacro:include filename="$(find andrzej_description)/urdf/andrzej_arms.xacro" />

File: urdf/andrzej_arms.xacro (robot description, xacro)
@@ -47,3 +47,16 @@
   <xacro:call macro="arm" arm_name="1"/>
   <xacro:call macro="arm" arm_name="2"/>
+  <xacro:macro name="servo" params="arm_name link_name">
+    <transmission name="arm_${arm_name}_tran_${link_name}">
+      <type>transmission_interface/SimpleTransmission</type>
+      <joint name="arm_${arm_name}_joint_${link_name}">
+        <hardwareInterface>PositionJointInterface</hardwareInterface>
+      </joint>
+      <actuator name="arm_${arm_name}_servo_${link_name}">
+        <hardwareInterface>PositionJointInterface</hardwareInterface>
+        <mechanicalReduction>1</mechanicalReduction>
+      </actuator>
+    </transmission>
+  </xacro:macro>
+  <xacro:call macro="servo" arm_name="1" link_name="1" />
 </robot>

File: urdf/andrzej_base.xacro (robot description, xacro)
@@ -1,4 +1,17 @@
 <?xml version="1.0"?>
 <robot name="andrzej" xmlns:xacro="http://ros.org/wiki/xacro">
+  <link name="base_footprint">
+   <visual>
+      <origin xyz="0 0 0" rpy="0 0 0" />
+      <geometry>
+        <box size="0.001 0.001 0.001" />
+      </geometry>
+    </visual>
+  </link>
+  <joint name="base_link_joint" type="fixed">
+    <origin xyz="0.0 0 0" rpy="0 0 0" />
+    <parent link="base_footprint"/>
+    <child link="base_link" />
+  </joint>
   <link name="base_link">
     <visual>
