Commit message: added ros control support for arm joints

File: andrzej_description/urdf/andrzej_arms.xacro (robot description, xacro)
@@ -23,4 +23,16 @@
     </joint>
   </xacro:macro>
+  <xacro:macro name="servo" params="arm_name link_name">
+    <transmission name="arm_${arm_name}_tran_${link_name}">
+      <type>transmission_interface/SimpleTransmission</type>
+      <joint name="arm_${arm_name}_joint_${link_name}">
+        <hardwareInterface>PositionJointInterface</hardwareInterface>
+      </joint>
+      <actuator name="arm_${arm_name}_servo_${link_name}">
+        <hardwareInterface>PositionJointInterface</hardwareInterface>
+        <mechanicalReduction>1</mechanicalReduction>
+      </actuator>
+    </transmission>
+  </xacro:macro>
   <xacro:macro name="arm_link" params="arm_name link_name">
     <link name="arm_${arm_name}_link_${link_name}">
@@ -35,4 +47,5 @@
       <child link="arm_${arm_name}_link_${link_name}"/>
     </joint>
+    <xacro:call macro="servo" arm_name="${arm_name}" link_name="${link_name}" />
   </xacro:macro>
   <xacro:macro name="arm" params="arm_name">
@@ -47,16 +60,3 @@
   <xacro:call macro="arm" arm_name="1"/>
   <xacro:call macro="arm" arm_name="2"/>
-  <xacro:macro name="servo" params="arm_name link_name">
-    <transmission name="arm_${arm_name}_tran_${link_name}">
-      <type>transmission_interface/SimpleTransmission</type>
-      <joint name="arm_${arm_name}_joint_${link_name}">
-        <hardwareInterface>PositionJointInterface</hardwareInterface>
-      </joint>
-      <actuator name="arm_${arm_name}_servo_${link_name}">
-        <hardwareInterface>PositionJointInterface</hardwareInterface>
-        <mechanicalReduction>1</mechanicalReduction>
-      </actuator>
-    </transmission>
-  </xacro:macro>
-  <xacro:call macro="servo" arm_name="1" link_name="1" />
 </robot>

Commit message: added grippers xacro

File: andrzej_description/urdf/andrzej_arms.xacro (robot description, xacro)
@@ -2,6 +2,7 @@
 <robot name="andrzej" xmlns:xacro="http://ros.org/wiki/xacro">
   <xacro:include filename="$(find andrzej_description)/urdf/andrzej_arms_spec.xacro" />
-  <xacro:macro name="arm_base" params="arm_name reflect">
-    <link name="arm_${arm_name}_link_0">
+  <xacro:include filename="$(find andrzej_description)/urdf/andrzej_gripper.xacro" />
+  <xacro:macro name="arm_base" params="arm reflect">
+    <link name="arm_${arm}_link_0">
       <visual>
         <geometry>
@@ -17,17 +18,17 @@
       <xacro:default_inertial mass="${arm_base_mass}"/>
     </link>
-    <joint name="platform_to_arm_${arm_name}" type="fixed">
+    <joint name="platform_to_arm_${arm}" type="fixed">
       <parent link="base_link"/>
-      <child link="arm_${arm_name}_link_0"/>
+      <child link="arm_${arm}_link_0"/>
       <origin xyz="${base_length*reflect/4} 0 ${(base_height+arm_base_height)/2}"/>
     </joint>
   </xacro:macro>
-  <xacro:macro name="servo" params="arm_name link_name">
-    <transmission name="arm_${arm_name}_tran_${link_name}">
+  <xacro:macro name="servo" params="arm link_name">
+    <transmission name="arm_${arm}_tran_${link_name}">
       <type>transmission_interface/SimpleTransmission</type>
-      <joint name="arm_${arm_name}_joint_${link_name}">
+      <joint name="arm_${arm}_joint_${link_name}">
         <hardwareInterface>PositionJointInterface</hardwareInterface>
       </joint>
-      <actuator name="arm_${arm_name}_servo_${link_name}">
+      <actuator name="arm_${arm}_servo_${link_name}">
         <hardwareInterface>PositionJointInterface</hardwareInterface>
         <mechanicalReduction>1</mechanicalReduction>
@@ -35,28 +36,29 @@
     </transmission>
   </xacro:macro>
-  <xacro:macro name="arm_link" params="arm_name link_name">
-    <link name="arm_${arm_name}_link_${link_name}">
+  <xacro:macro name="arm_link" params="arm link_name">
+    <link name="arm_${arm}_link_${link_name}">
       <visual>
-        <xacro:call macro="arm_${arm_name}_link_${link_name}_visual"/>
+        <xacro:call macro="arm_${arm}_link_${link_name}_visual"/>
       </visual>
-      <xacro:call macro="arm_${arm_name}_link_${link_name}_inertia"/>
+      <xacro:call macro="arm_${arm}_link_${link_name}_inertia"/>
     </link>
-    <joint name="arm_${arm_name}_joint_${link_name}" type="revolute">
-      <xacro:call macro="arm_${arm_name}_joint_${link_name}_spec"/>
-      <parent link="arm_${arm_name}_link_${link_name-1}"/>
-      <child link="arm_${arm_name}_link_${link_name}"/>
+    <joint name="arm_${arm}_joint_${link_name}" type="revolute">
+      <xacro:call macro="arm_${arm}_joint_${link_name}_spec"/>
+      <parent link="arm_${arm}_link_${link_name-1}"/>
+      <child link="arm_${arm}_link_${link_name}"/>
     </joint>
-    <xacro:call macro="servo" arm_name="${arm_name}" link_name="${link_name}" />
+    <xacro:call macro="servo" arm="${arm}" link_name="${link_name}" />
   </xacro:macro>
-  <xacro:macro name="arm" params="arm_name">
-    <xacro:arm_link arm_name="${arm_name}" link_name="1"/>
-    <xacro:arm_link arm_name="${arm_name}" link_name="2"/>
-    <xacro:arm_link arm_name="${arm_name}" link_name="3"/>
-    <xacro:arm_link arm_name="${arm_name}" link_name="4"/>
-    <xacro:arm_link arm_name="${arm_name}" link_name="5"/>
+  <xacro:macro name="arm" params="arm_id">
+    <xacro:arm_link arm="${arm_id}" link_name="1"/>
+    <xacro:arm_link arm="${arm_id}" link_name="2"/>
+    <xacro:arm_link arm="${arm_id}" link_name="3"/>
+    <xacro:arm_link arm="${arm_id}" link_name="4"/>
+    <xacro:arm_link arm="${arm_id}" link_name="5"/>
+    <xacro:gripper arm="${arm_id}"/>
   </xacro:macro>
-  <xacro:call macro="arm_base" arm_name="1" reflect="1" />
-  <xacro:call macro="arm_base" arm_name="2" reflect="-1" />
-  <xacro:call macro="arm" arm_name="1"/>
-  <xacro:call macro="arm" arm_name="2"/>
+  <xacro:call macro="arm_base" arm="1" reflect="1" />
+  <xacro:call macro="arm_base" arm="2" reflect="-1" />
+  <xacro:call macro="arm" arm_id="1"/>
+  <xacro:call macro="arm" arm_id="2"/>
 </robot>

Commit message: fixed arm 1 dimensions, added more visuals

File: andrzej_description/urdf/andrzej_arms.xacro (robot description, xacro)
@@ -7,11 +7,18 @@
       <visual>
         <geometry>
-          <box size="${arm_base_length} ${arm_base_width} ${arm_base_height}"/>
+          <box size=".15 .15 .035"/>
         </geometry>
+        <origin xyz="0 0 ${(.035)/2}"/>
         <material name="orange"/>
+      </visual>
+      <visual>
+        <geometry>
+          <box size=".1 .1 .02"/>
+        </geometry>
+        <origin xyz="0 0 0.045"/>
       </visual>
       <collision>
         <geometry>
-          <box size="${arm_base_length} ${arm_base_width} ${arm_base_height}"/>
+          <box size=".15 .15 .035"/>
         </geometry>
       </collision>
@@ -21,5 +28,5 @@
       <parent link="base_link"/>
       <child link="arm_${arm}_link_0"/>
-      <origin xyz="${base_length*reflect/4} 0 ${(base_height+arm_base_height)/2}"/>
+      <origin xyz="${0.125*reflect} 0 ${base_height/2}"/>
     </joint>
   </xacro:macro>
@@ -38,7 +45,5 @@
   <xacro:macro name="arm_link" params="arm link_name">
     <link name="arm_${arm}_link_${link_name}">
-      <visual>
-        <xacro:call macro="arm_${arm}_link_${link_name}_visual"/>
-      </visual>
+      <xacro:call macro="arm_${arm}_link_${link_name}_visual"/>
       <xacro:call macro="arm_${arm}_link_${link_name}_inertia"/>
     </link>

File: andrzej_description/urdf/andrzej_arms_spec.xacro (robot description, xacro)
@@ -1,127 +1,220 @@
 <?xml version="1.0"?>
 <robot name="andrzej" xmlns:xacro="http://ros.org/wiki/xacro">
-  <xacro:property name="arm_base_length" value=".2" />
-  <xacro:property name="arm_base_width" value=".2" />
-  <xacro:property name="arm_base_height" value=".05" />
+  <xacro:property name="arm_base_length" value=".15" />
+  <xacro:property name="arm_base_width" value=".15" />
+  <xacro:property name="arm_base_height" value=".055" />
   <xacro:macro name="arm_1_link_1_visual">
-    <geometry>
-          <box size=".1 .05 .05"/>
-    </geometry>
-    <origin xyz="0 0 0.025"/>
-    <material name="green"/>
+    <visual>
+      <geometry>
+          <cylinder radius="0.0375" length="0.02"/>
+      </geometry>
+      <origin xyz="0 0 -0.01"/>
+      <material name="gray"/>
+    </visual>
+    <visual>
+      <geometry>
+          <box size=".1 .1 .01"/>
+      </geometry>
+      <origin xyz="0 0 0.005"/>
+    </visual>
+    <visual>
+      <geometry>
+          <box size=".05 .05 .01"/>
+      </geometry>
+      <origin xyz="0.075 0 0.005"/>
+    </visual>
+    <visual>
+      <geometry>
+          <box size=".03 .025 .04"/>
+      </geometry>
+      <origin xyz="0.075 0 0.03"/>
+    </visual>
+    <visual>
+      <geometry>
+          <box size=".03 .025 .04"/>
+      </geometry>
+      <origin xyz="0 0 0.03"/>
+    </visual>
   </xacro:macro>
   <xacro:macro name="arm_1_joint_1_spec">
     <axis xyz="0 0 1"/>
     <limit effort="1000.0" lower="-.67" upper="2.67" velocity="0.5"/>
-    <origin xyz="0 0 0"/>
+    <origin xyz="0 0 .07"/>
   </xacro:macro>
   <xacro:macro name="arm_1_link_2_visual">
-    <geometry>
-      <box size=".1 .05 .2"/>
-    </geometry>
-    <origin xyz="0 0 .1"/>
-    <material name="gray"/>
+    <visual>
+      <geometry>
+        <box size=".005 .05 ${.2+.02}"/>
+      </geometry>
+      <origin xyz="-0.03 0 .1"/>
+      <material name="orange"/>
+    </visual>
+    <visual>
+      <geometry>
+        <box size=".005 .05 ${.2+.02}"/>
+      </geometry>
+      <origin xyz="0.03 0 .1"/>
+      <material name="orange"/>
+    </visual>
+    <visual>
+      <geometry>
+        <box size=".06 .02 .04"/>
+      </geometry>
+      <origin xyz="0 0 .1"/>
+      <material name="orange"/>
+    </visual>
   </xacro:macro>
   <xacro:macro name="arm_1_joint_2_spec">
+    <axis xyz="1 0 0"/>
+    <limit effort="1000.0" lower="-1.47" upper="1.87" velocity="0.5"/>
+    <origin xyz="0 0 0.04"/>
+  </xacro:macro>
+  <xacro:macro name="arm_1_link_3_visual">
+    <visual>
+      <geometry>
+        <box size=".005 .03 .18"/>
+      </geometry>
+      <origin xyz="-.015 0 .05"/>
+      <material name="orange"/>
+    </visual>
+    <visual>
+      <geometry>
+        <box size=".005 .03 .18"/>
+      </geometry>
+      <origin xyz=".015 0 .05"/>
+      <material name="orange"/>
+    </visual>
+    <visual>
+      <geometry>
+        <box size=".045 .02 .05"/>
+      </geometry>
+      <origin xyz="0 0 -0.01"/>
+      <material name="orange"/>
+    </visual>
+    <visual>
+      <geometry>
+        <box size=".02 .05 .045"/>
+      </geometry>
+      <origin xyz="0 0 ${.14-.045/2}"/>
+      <material name="orange"/>
+    </visual>
+  </xacro:macro>
+  <xacro:macro name="arm_1_joint_3_spec">
+    <axis xyz="1 0 0"/>
+    <limit effort="1000.0" lower="-.87" upper="2.47" velocity="0.5"/>
+    <origin xyz="0 0 .19"/>
+  </xacro:macro>
+  <xacro:macro name="arm_1_link_4_visual">
+    <visual>
+      <geometry>
+        <box size=".05 .02 .06"/>
+      </geometry>
+      <origin xyz="0 0 .03"/>
+      <material name="gray"/>
+    </visual>
+  </xacro:macro>
+  <xacro:macro name="arm_1_joint_4_spec">
+    <axis xyz="0 0 1"/>
+    <limit effort="1000.0" lower="-1.67" upper="1.67" velocity="0.5"/>
+    <origin xyz="0 0 .14"/>
+  </xacro:macro>
+  <xacro:macro name="arm_1_link_5_visual">
+    <visual>
+      <geometry>
+        <box size=".005 .03 .05"/>
+      </geometry>
+      <origin xyz="-.0325 0 .005"/>
+      <material name="gray"/>
+    </visual>
+    <visual>
+      <geometry>
+        <box size=".005 .03 .05"/>
+      </geometry>
+      <origin xyz=".0325 0 .005"/>
+      <material name="gray"/>
+    </visual>
+    <visual>
+      <geometry>
+        <box size=".065 .03 .005"/>
+      </geometry>
+      <origin xyz="0 0 .03"/>
+      <material name="gray"/>
+    </visual>
+  </xacro:macro>
+  <xacro:macro name="arm_1_joint_5_spec">
+    <axis xyz="1 0 0"/>
+    <limit effort="1000.0" lower="-1.67" upper="1.67" velocity="0.5"/>
+    <origin xyz="0 0 .05"/>
+  </xacro:macro>
+  <xacro:macro name="arm_2_link_1_visual">
+    <visual>
+      <geometry>
+            <box size=".1 .05 .05"/>
+      </geometry>
+      <origin xyz="0 0 0.025"/>
+      <material name="gray"/>
+    </visual>
+  </xacro:macro>
+  <xacro:macro name="arm_2_joint_1_spec">
+    <axis xyz="0 0 1"/>
+    <limit effort="1000.0" lower="-.67" upper="2.67" velocity="0.5"/>
+    <origin xyz="0 0 .055"/>
+  </xacro:macro>
+  <xacro:macro name="arm_2_link_2_visual">
+    <visual>
+      <geometry>
+        <box size=".1 .05 .2"/>
+      </geometry>
+      <origin xyz="0 0 .1"/>
+      <material name="gray"/>
+    </visual>
+  </xacro:macro>
+  <xacro:macro name="arm_2_joint_2_spec">
     <axis xyz="1 0 0"/>
     <limit effort="1000.0" lower="-1.47" upper="1.87" velocity="0.5"/>
     <origin xyz="0 0 0.05"/>
   </xacro:macro>
-  <xacro:macro name="arm_1_link_3_visual">
-    <geometry>
-      <box size=".1 .05 .2"/>
-    </geometry>
-    <origin xyz="0 0 .1"/>
-    <material name="orange"/>
-  </xacro:macro>
-  <xacro:macro name="arm_1_joint_3_spec">
+  <xacro:macro name="arm_2_link_3_visual">
+    <visual>
+      <geometry>
+        <box size=".1 .05 .2"/>
+      </geometry>
+      <origin xyz="0 0 .1"/>
+      <material name="orange"/>
+    </visual>
+  </xacro:macro>
+  <xacro:macro name="arm_2_joint_3_spec">
     <axis xyz="1 0 0"/>
     <limit effort="1000.0" lower="-.87" upper="2.47" velocity="0.5"/>
     <origin xyz="0 0 .3"/>
   </xacro:macro>
-  <xacro:macro name="arm_1_link_4_visual">
-    <geometry>
-      <box size=".1 .05 .05"/>
-    </geometry>
-    <origin xyz="0 0 .025"/>
-    <material name="gray"/>
-  </xacro:macro>
-  <xacro:macro name="arm_1_joint_4_spec">
+  <xacro:macro name="arm_2_link_4_visual">
+    <visual>
+      <geometry>
+        <box size=".1 .05 .05"/>
+      </geometry>
+      <origin xyz="0 0 .025"/>
+      <material name="gray"/>
+    </visual>
+  </xacro:macro>
+  <xacro:macro name="arm_2_joint_4_spec">
     <axis xyz="0 0 1"/>
     <limit effort="1000.0" lower="-1.67" upper="1.67" velocity="0.5"/>
     <origin xyz="0 0 .2"/>
   </xacro:macro>
-  <xacro:macro name="arm_1_link_5_visual">
-    <geometry>
-      <box size=".1 .05 .05"/>
-    </geometry>
-    <origin xyz="0 0 .025"/>
-    <material name="gray"/>
-  </xacro:macro>
-  <xacro:macro name="arm_1_joint_5_spec">
+  <xacro:macro name="arm_2_link_5_visual">
+    <visual>
+      <geometry>
+        <box size=".1 .05 .05"/>
+      </geometry>
+      <origin xyz="0 0 .025"/>
+      <material name="gray"/>
+    </visual>
+  </xacro:macro>
+  <xacro:macro name="arm_2_joint_5_spec">
     <axis xyz="1 0 0"/>
     <limit effort="1000.0" lower="-1.67" upper="1.67" velocity="0.5"/>
     <origin xyz="0 0 .05"/>
   </xacro:macro>
-  <xacro:macro name="arm_2_link_1_visual">
-    <geometry>
-          <box size=".1 .05 .05"/>
-    </geometry>
-    <origin xyz="0 0 0.025"/>
-    <material name="green"/>
-  </xacro:macro>
-  <xacro:macro name="arm_2_joint_1_spec">
-    <axis xyz="0 0 1"/>
-    <limit effort="1000.0" lower="-.67" upper="2.67" velocity="0.5"/>
-    <origin xyz="0 0 0"/>
-  </xacro:macro>
-  <xacro:macro name="arm_2_link_2_visual">
-    <geometry>
-      <box size=".1 .05 .2"/>
-    </geometry>
-    <origin xyz="0 0 .1"/>
-    <material name="gray"/>
-  </xacro:macro>
-  <xacro:macro name="arm_2_joint_2_spec">
-    <axis xyz="1 0 0"/>
-    <limit effort="1000.0" lower="-1.47" upper="1.87" velocity="0.5"/>
-    <origin xyz="0 0 0.05"/>
-  </xacro:macro>
-  <xacro:macro name="arm_2_link_3_visual">
-    <geometry>
-      <box size=".1 .05 .2"/>
-    </geometry>
-    <origin xyz="0 0 .1"/>
-    <material name="orange"/>
-  </xacro:macro>
-  <xacro:macro name="arm_2_joint_3_spec">
-    <axis xyz="1 0 0"/>
-    <limit effort="1000.0" lower="-.87" upper="2.47" velocity="0.5"/>
-    <origin xyz="0 0 .3"/>
-  </xacro:macro>
-  <xacro:macro name="arm_2_link_4_visual">
-    <geometry>
-      <box size=".1 .05 .05"/>
-    </geometry>
-    <origin xyz="0 0 .025"/>
-    <material name="gray"/>
-  </xacro:macro>
-  <xacro:macro name="arm_2_joint_4_spec">
-    <axis xyz="0 0 1"/>
-    <limit effort="1000.0" lower="-1.67" upper="1.67" velocity="0.5"/>
-    <origin xyz="0 0 .2"/>
-  </xacro:macro>
-  <xacro:macro name="arm_2_link_5_visual">
-    <geometry>
-      <box size=".1 .05 .05"/>
-    </geometry>
-    <origin xyz="0 0 .025"/>
-    <material name="gray"/>
-  </xacro:macro>
-  <xacro:macro name="arm_2_joint_5_spec">
-    <axis xyz="1 0 0"/>
-    <limit effort="1000.0" lower="-1.67" upper="1.67" velocity="0.5"/>
-    <origin xyz="0 0 .05"/>
-  </xacro:macro>
   <xacro:macro name="arm_1_link_1_inertia">
     <inertial>
