Commit message: fixed arm2 dimensions and visuals

File: andrzej_description/urdf/andrzej_arms_spec.xacro (robot description, xacro)
@@ -45,5 +45,5 @@
     <visual>
       <geometry>
-        <box size=".005 .05 ${.2+.02}"/>
+        <box size=".005 .05 ${.2+.01}"/>
       </geometry>
       <origin xyz="-0.03 0 .1"/>
@@ -52,5 +52,5 @@
     <visual>
       <geometry>
-        <box size=".005 .05 ${.2+.02}"/>
+        <box size=".005 .05 ${.2+.01}"/>
       </geometry>
       <origin xyz="0.03 0 .1"/>
@@ -68,5 +68,5 @@
     <axis xyz="1 0 0"/>
     <limit effort="1000.0" lower="-1.47" upper="1.87" velocity="0.5"/>
-    <origin xyz="0 0 0.04"/>
+    <origin xyz="0 0 0.03"/>
   </xacro:macro>
   <xacro:macro name="arm_1_link_3_visual">
@@ -150,8 +150,32 @@
     <visual>
       <geometry>
-            <box size=".1 .05 .05"/>
-      </geometry>
-      <origin xyz="0 0 0.025"/>
-      <material name="gray"/>
+          <cylinder radius="0.0375" length="0.02"/>
+      </geometry>
+      <origin xyz="0 0 -0.01"/>
+      <material name="gray"/>
+    </visual>
+    <visual>
+      <geometry>
+          <box size=".1 .1 .01"/>
+      </geometry>
+      <origin xyz="0 0 0.005"/>
+    </visual>
+    <visual>
+      <geometry>
+          <box size=".05 .05 .01"/>
+      </geometry>
+      <origin xyz="-0.075 0 0.005"/>
+    </visual>
+    <visual>
+      <geometry>
+          <box size=".03 .025 .04"/>
+      </geometry>
+      <origin xyz="-0.075 0 0.03"/>
+    </visual>
+    <visual>
+      <geometry>
+          <box size=".03 .025 .04"/>
+      </geometry>
+      <origin xyz="0 0 0.03"/>
     </visual>
   </xacro:macro>
@@ -159,13 +183,27 @@
     <axis xyz="0 0 1"/>
     <limit effort="1000.0" lower="-.67" upper="2.67" velocity="0.5"/>
-    <origin xyz="0 0 .055"/>
+    <origin xyz="0 0 .07"/>
   </xacro:macro>
   <xacro:macro name="arm_2_link_2_visual">
     <visual>
       <geometry>
-        <box size=".1 .05 .2"/>
-      </geometry>
-      <origin xyz="0 0 .1"/>
-      <material name="gray"/>
+        <box size=".005 .05 ${.14+.01}"/>
+      </geometry>
+      <origin xyz="-0.03 0 .075"/>
+      <material name="orange"/>
+    </visual>
+    <visual>
+      <geometry>
+        <box size=".005 .05 ${.14+.01}"/>
+      </geometry>
+      <origin xyz="0.03 0 .075"/>
+      <material name="orange"/>
+    </visual>
+    <visual>
+      <geometry>
+        <box size=".06 .02 .04"/>
+      </geometry>
+      <origin xyz="0 0 .075"/>
+      <material name="orange"/>
     </visual>
   </xacro:macro>
@@ -173,12 +211,33 @@
     <axis xyz="1 0 0"/>
     <limit effort="1000.0" lower="-1.47" upper="1.87" velocity="0.5"/>
-    <origin xyz="0 0 0.05"/>
+    <origin xyz="0 0 0.03"/>
   </xacro:macro>
   <xacro:macro name="arm_2_link_3_visual">
     <visual>
       <geometry>
-        <box size=".1 .05 .2"/>
-      </geometry>
-      <origin xyz="0 0 .1"/>
+        <box size=".005 .03 .14"/>
+      </geometry>
+      <origin xyz="-.015 0 .06"/>
+      <material name="orange"/>
+    </visual>
+    <visual>
+      <geometry>
+        <box size=".005 .03 .14"/>
+      </geometry>
+      <origin xyz=".015 0 .06"/>
+      <material name="orange"/>
+    </visual>
+    <visual>
+      <geometry>
+        <box size=".045 .02 .05"/>
+      </geometry>
+      <origin xyz="0 0 0.02"/>
+      <material name="orange"/>
+    </visual>
+    <visual>
+      <geometry>
+        <box size=".02 .05 .045"/>
+      </geometry>
+      <origin xyz="0 0 ${.13-.045/2}"/>
       <material name="orange"/>
     </visual>
@@ -187,12 +246,12 @@
     <axis xyz="1 0 0"/>
     <limit effort="1000.0" lower="-.87" upper="2.47" velocity="0.5"/>
-    <origin xyz="0 0 .3"/>
+    <origin xyz="0 0 .14"/>
   </xacro:macro>
   <xacro:macro name="arm_2_link_4_visual">
     <visual>
       <geometry>
-        <box size=".1 .05 .05"/>
-      </geometry>
-      <origin xyz="0 0 .025"/>
+        <box size=".05 .02 .06"/>
+      </geometry>
+      <origin xyz="0 0 .03"/>
       <material name="gray"/>
     </visual>
@@ -201,12 +260,26 @@
     <axis xyz="0 0 1"/>
     <limit effort="1000.0" lower="-1.67" upper="1.67" velocity="0.5"/>
-    <origin xyz="0 0 .2"/>
+    <origin xyz="0 0 .13"/>
   </xacro:macro>
   <xacro:macro name="arm_2_link_5_visual">
     <visual>
       <geometry>
-        <box size=".1 .05 .05"/>
-      </geometry>
-      <origin xyz="0 0 .025"/>
+        <box size=".005 .03 .05"/>
+      </geometry>
+      <origin xyz="-.0325 0 .005"/>
+      <material name="gray"/>
+    </visual>
+    <visual>
+      <geometry>
+        <box size=".005 .03 .05"/>
+      </geometry>
+      <origin xyz=".0325 0 .005"/>
+      <material name="gray"/>
+    </visual>
+    <visual>
+      <geometry>
+        <box size=".065 .03 .005"/>
+      </geometry>
+      <origin xyz="0 0 .03"/>
       <material name="gray"/>
     </visual>
