Commit message: gripper controller - separate for each finger for now

File: andrzej_description/urdf/andrzej.xacro (robot description, xacro)
@@ -11,4 +11,6 @@
   <xacro:property name="wheel_mass" value="0.3" />
   <xacro:property name="arm_base_mass" value="0.2" />
+  <xacro:property name="gripper_base_mass" value="0.03" />
+  <xacro:property name="gripper_finger_mass" value="0.02" />
   <xacro:include filename="$(find andrzej_description)/urdf/materials.xacro" />
   <xacro:macro name="default_inertial" params="mass">

File: andrzej_description/urdf/andrzej_gripper.xacro (robot description, xacro)
@@ -17,4 +17,5 @@
       <material name="black"/>
     </visual>
+    <xacro:default_inertial mass="${gripper_finger_mass}"/>
   </link>
   <joint name="arm_${arm}_finger_${suffix}_joint" type="revolute">
@@ -25,4 +26,14 @@
     <child link="arm_${arm}_finger_${suffix}_link"/>
   </joint>
+  <transmission name="arm_${arm}_finger_${suffix}_trans">
+    <type>transmission_interface/SimpleTransmission</type>
+    <joint name="arm_${arm}_finger_${suffix}_joint">
+      <hardwareInterface>PositionJointInterface</hardwareInterface>
+    </joint>
+    <actuator name="arm_${arm}_gripper_servo">
+      <hardwareInterface>PositionJointInterface</hardwareInterface>
+      <mechanicalReduction>1</mechanicalReduction>
+    </actuator>
+  </transmission>
 </xacro:macro>
 <xacro:macro name="gripper" params="arm" >
@@ -35,4 +46,5 @@
       <material name="gray"/>
     </visual>
+    <xacro:default_inertial mass="${gripper_base_mass}"/>
   </link>
   <joint name="arm_${arm}_gripper_base_joint" type="fixed">

Commit message: added head pole, fixed base dimensions

File: andrzej_description/urdf/andrzej.xacro (robot description, xacro)
@@ -2,9 +2,9 @@
 <robot name="andrzej" xmlns:xacro="http://ros.org/wiki/xacro">
   <!-- Dimensions -->
-  <xacro:property name="base_width" value=".4" />
-  <xacro:property name="base_length" value=".6" />
-  <xacro:property name="base_height" value=".1" />
+  <xacro:property name="base_width" value=".3" />
+  <xacro:property name="base_length" value=".47" />
+  <xacro:property name="base_height" value=".09" />
   <xacro:property name="wheel_diam" value=".1" />
-  <xacro:property name="wheel_width" value=".04" />
+  <xacro:property name="wheel_width" value=".05" />
   <!-- Masses-->
   <xacro:property name="base_mass" value="5" />
@@ -13,4 +13,5 @@
   <xacro:property name="gripper_base_mass" value="0.03" />
   <xacro:property name="gripper_finger_mass" value="0.02" />
+  <xacro:property name="head_pole_mass" value="0.3" />
   <xacro:include filename="$(find andrzej_description)/urdf/materials.xacro" />
   <xacro:macro name="default_inertial" params="mass">
@@ -23,3 +24,4 @@
   <xacro:include filename="$(find andrzej_description)/urdf/andrzej_base.xacro" />
   <xacro:include filename="$(find andrzej_description)/urdf/andrzej_arms.xacro" />
+  <xacro:include filename="$(find andrzej_description)/urdf/andrzej_head.xacro" />
 </robot>

File: andrzej_description/urdf/andrzej_base.xacro (robot description, xacro)
@@ -49,5 +49,7 @@
       <parent link="base_link"/>
       <child link="${prefix}_wheel"/>
-      <origin xyz="${base_length*reflect_x/3} ${(base_width/2+wheel_width/2)*reflect_y} ${-base_height/2+wheel_diam/4}" rpy="0 0 0"/>
+      <origin xyz="${0.17*reflect_x}
+                   ${(base_width/2 + wheel_width/2 + .02)*reflect_y}
+                   ${-base_height/2 + 0.02}" rpy="0 0 0"/>
     </joint>
   </xacro:macro>

Commit message: added head pan tilt urdf

File: andrzej_description/urdf/andrzej.xacro (robot description, xacro)
@@ -1,4 +1,4 @@
 <?xml version="1.0"?>
-<robot name="andrzej" xmlns:xacro="http://ros.org/wiki/xacro">
+<robot name="andrzej" xmlns:xacro="http://www.ros.org/wiki/xacro">
   <!-- Dimensions -->
   <xacro:property name="base_width" value=".3" />

File: andrzej_description/urdf/andrzej_arms.xacro (robot description, xacro)
@@ -1,4 +1,4 @@
 <?xml version="1.0"?>
-<robot name="andrzej" xmlns:xacro="http://ros.org/wiki/xacro">
+<robot name="andrzej" xmlns:xacro="http://www.ros.org/wiki/xacro">
   <xacro:include filename="$(find andrzej_description)/urdf/andrzej_arms_spec.xacro" />
   <xacro:include filename="$(find andrzej_description)/urdf/andrzej_gripper.xacro" />

File: andrzej_description/urdf/andrzej_arms_spec.xacro (robot description, xacro)
@@ -1,4 +1,4 @@
 <?xml version="1.0"?>
-<robot name="andrzej" xmlns:xacro="http://ros.org/wiki/xacro">
+<robot name="andrzej" xmlns:xacro="http://www.ros.org/wiki/xacro">
   <xacro:property name="arm_base_length" value=".15" />
   <xacro:property name="arm_base_width" value=".15" />

File: andrzej_description/urdf/andrzej_base.xacro (robot description, xacro)
@@ -1,4 +1,4 @@
 <?xml version="1.0"?>
-<robot name="andrzej" xmlns:xacro="http://ros.org/wiki/xacro">
+<robot name="andrzej" xmlns:xacro="http://www.ros.org/wiki/xacro">
   <link name="base_footprint">
    <visual>

File: andrzej_description/urdf/andrzej_gripper.xacro (robot description, xacro)
@@ -1,4 +1,4 @@
 <?xml version="1.0"?>
-<robot name="andrzej" xmlns:xacro="http://ros.org/wiki/xacro">
+<robot name="andrzej" xmlns:xacro="http://www.ros.org/wiki/xacro">
 <xacro:macro name="finger" params="arm suffix reflect" >
   <link name="arm_${arm}_finger_${suffix}_link">

File: andrzej_description/urdf/andrzej_head.xacro (robot description, xacro)
@@ -1,4 +1,4 @@
 <?xml version="1.0"?>
-<robot name="andrzej" xmlns:xacro="http://ros.org/wiki/xacro">
+<robot name="andrzej" xmlns:xacro="http://www.ros.org/wiki/xacro">
 <xacro:property name="head_pole_width" value=".025" />
 <xacro:property name="head_pole_height" value=".5" />
@@ -9,5 +9,5 @@
     </geometry>
     <origin xyz="0 0 ${head_pole_height/2}"/>
-    <material name="green"/>
+    <material name="gray"/>
   </visual>
   <visual>
@@ -16,5 +16,4 @@
     </geometry>
     <origin xyz="0 0 0.005"/>
-    <material name="green"/>
   </visual>
   <xacro:default_inertial mass="${head_pole_mass}"/>
@@ -25,3 +24,70 @@
   <origin xyz="0 ${base_width/2 - head_pole_width} ${base_height/2}"/>
 </joint>
+<link name="head_base_link">
+  <visual>
+    <geometry>
+      <box size=".02 .06 .05"/>
+    </geometry>
+    <origin xyz="0 0 -.02"/>
+    <material name="black"/>
+  </visual>
+  <xacro:default_inertial mass=".1"/>
+</link>
+<joint name="head_base_joint" type="fixed">
+  <parent link="head_pole"/>
+  <child link="head_base_link"/>
+  <origin xyz="0 ${head_pole_width/2 + .03} ${head_pole_height}"/>
+</joint>
+<link name="head_pan_link">
+  <visual>
+    <geometry>
+      <box size=".04 .065 .03"/>
+    </geometry>
+    <origin xyz="-.01 0 .015"/>
+    <material name="black"/>
+  </visual>
+  <xacro:default_inertial mass=".1"/>
+</link>
+<joint name="head_pan_joint" type="revolute">
+  <axis xyz="0 0 1"/>
+  <limit effort="1000.0" lower="-.67" upper="2.67" velocity="0.5"/>
+  <origin xyz="0 -.01 .015"/>
+  <parent link="head_base_link"/>
+  <child link="head_pan_link"/>
+</joint>
+<link name="head_tilt_link">
+  <visual>
+    <geometry>
+      <box size=".005 .0275 .05"/>
+    </geometry>
+    <origin xyz="-.0375 0 .01"/>
+    <material name="black"/>
+  </visual>
+  <visual>
+    <geometry>
+      <box size=".005 .0275 .05"/>
+    </geometry>
+    <origin xyz=".0175 0 .01"/>
+  </visual>
+  <visual>
+    <geometry>
+      <box size=".055 .0275 .005"/>
+    </geometry>
+    <origin xyz="-.01 0 .035"/>
+  </visual>
+  <xacro:default_inertial mass=".1"/>
+</link>
+<joint name="head_tilt_joint" type="revolute">
+  <axis xyz="1 0 0"/>
+  <limit effort="1000.0" lower="-.67" upper="2.67" velocity="0.5"/>
+  <origin xyz="0 -.01 .015"/>
+  <parent link="head_pan_link"/>
+  <child link="head_tilt_link"/>
+</joint>
+<!--
+<xacro:include filename="$(find hector_sensors_description)/urdf/asus_camera.urdf.xacro"/>
+<xacro:asus_camera name="head_camera" parent="head_tilt_link">
+  <origin xyz="0 0 .05" rpy="0 0 -${pi/2}" />
+</xacro:asus_camera>
+-->
 </robot>
