Commit message: fixed gripper dimensions and visuals

File: andrzej_description/urdf/andrzej_gripper.xacro (robot description, xacro)
@@ -5,22 +5,22 @@
     <visual>
       <geometry>
-        <box size=".075 .02 .05"/>
+        <box size=".01 .005 .08"/>
       </geometry>
-      <origin xyz=".0375 .02 0"/>
+      <origin xyz="0 ${reflect*0.025} .0325"/>
       <material name="gray"/>
     </visual>
     <visual>
       <geometry>
-        <box size=".04 .01 .05"/>
+        <box size=".02 .025 .04"/>
       </geometry>
-      <origin xyz=".055 .005 0"/>
-      <material name="black"/>
+      <origin xyz="-0.005 ${reflect*0.01} .045"/>
+      <material name="gray"/>
     </visual>
     <xacro:default_inertial mass="${gripper_finger_mass}"/>
   </link>
   <joint name="arm_${arm}_finger_${suffix}_joint" type="revolute">
-    <axis xyz="0 0 1"/>
+    <axis xyz="0 1 0"/>
     <limit effort="1000.0" lower="0.0" upper="0.548" velocity="0.5"/>
-    <origin rpy="0 ${-pi/2} ${reflect*pi/2}" xyz="0 0 0.02"/>
+    <origin rpy="0 0 ${reflect*pi/2-pi/2}" xyz="${reflect*0.015} 0 0"/>
     <parent link="arm_${arm}_gripper_base"/>
     <child link="arm_${arm}_finger_${suffix}_link"/>
@@ -41,8 +41,8 @@
     <visual>
       <geometry>
-        <box size=".1 .05 .02"/>
+        <box size=".045 .04 .02"/>
       </geometry>
-      <origin xyz="0 0 .01"/>
-      <material name="gray"/>
+      <origin xyz="0 0 .005"/>
+      <material name="black"/>
     </visual>
     <xacro:default_inertial mass="${gripper_base_mass}"/>

Commit message: fingers as mimic joints

File: andrzej_description/urdf/andrzej_gripper.xacro (robot description, xacro)
@@ -37,4 +37,31 @@
   </transmission>
 </xacro:macro>
+<xacro:macro name="finger_mimic" params="arm suffix mimic reflect" >
+  <link name="arm_${arm}_finger_${suffix}_link">
+    <visual>
+      <geometry>
+        <box size=".01 .005 .08"/>
+      </geometry>
+      <origin xyz="0 ${reflect*0.025} .0325"/>
+      <material name="gray"/>
+    </visual>
+    <visual>
+      <geometry>
+        <box size=".02 .025 .04"/>
+      </geometry>
+      <origin xyz="-0.005 ${reflect*0.01} .045"/>
+      <material name="gray"/>
+    </visual>
+    <xacro:default_inertial mass="${gripper_finger_mass}"/>
+  </link>
+  <joint name="arm_${arm}_finger_${suffix}_joint" type="revolute">
+    <axis xyz="0 1 0"/>
+    <limit effort="1000.0" lower="0.0" upper="0.548" velocity="0.5"/>
+    <origin rpy="0 0 ${reflect*pi/2-pi/2}" xyz="${reflect*0.015} 0 0"/>
+    <parent link="arm_${arm}_gripper_base"/>
+    <child link="arm_${arm}_finger_${suffix}_link"/>
+		<mimic joint="arm_${arm}_finger_${mimic}_joint" multiplier="1" offset="0"/>
+  </joint>
+</xacro:macro>
 <xacro:macro name="gripper" params="arm" >
   <link name="arm_${arm}_gripper_base">
@@ -54,5 +81,5 @@
   </joint>
   <xacro:call macro="finger" arm="${arm}" suffix="left" reflect="1"/>
-  <xacro:call macro="finger" arm="${arm}" suffix="right" reflect="-1"/>
+  <xacro:call macro="finger_mimic" arm="${arm}" suffix="right" mimic="left" reflect="-1"/>
 </xacro:macro>
 </robot>

Commit message: control: gripper hw iface

File: andrzej_description/urdf/andrzej_gripper.xacro (robot description, xacro)
@@ -1,5 +1,5 @@
 <?xml version="1.0"?>
 <robot name="andrzej" xmlns:xacro="http://www.ros.org/wiki/xacro">
-<xacro:macro name="finger" params="arm suffix reflect" >
+<xacro:macro name="finger_link" params="arm suffix reflect" >
   <link name="arm_${arm}_finger_${suffix}_link">
     <visual>
@@ -19,14 +19,16 @@
     <xacro:default_inertial mass="${gripper_finger_mass}"/>
   </link>
-  <joint name="arm_${arm}_finger_${suffix}_joint" type="revolute">
+</xacro:macro>
+<xacro:macro name="gripper_joint" params="arm reflect" >
+  <joint name="arm_${arm}_gripper_joint" type="revolute">
     <axis xyz="0 1 0"/>
     <limit effort="1000.0" lower="0.0" upper="0.548" velocity="0.5"/>
     <origin rpy="0 0 ${reflect*pi/2-pi/2}" xyz="${reflect*0.015} 0 0"/>
     <parent link="arm_${arm}_gripper_base"/>
-    <child link="arm_${arm}_finger_${suffix}_link"/>
+    <child link="arm_${arm}_finger_left_link"/>
   </joint>
-  <transmission name="arm_${arm}_finger_${suffix}_trans">
+  <transmission name="arm_${arm}_finger_left_trans">
     <type>transmission_interface/SimpleTransmission</type>
-    <joint name="arm_${arm}_finger_${suffix}_joint">
+    <joint name="arm_${arm}_gripper_joint">
       <hardwareInterface>PositionJointInterface</hardwareInterface>
     </joint>
@@ -36,30 +38,11 @@
     </actuator>
   </transmission>
-</xacro:macro>
-<xacro:macro name="finger_mimic" params="arm suffix mimic reflect" >
-  <link name="arm_${arm}_finger_${suffix}_link">
-    <visual>
-      <geometry>
-        <box size=".01 .005 .08"/>
-      </geometry>
-      <origin xyz="0 ${reflect*0.025} .0325"/>
-      <material name="gray"/>
-    </visual>
-    <visual>
-      <geometry>
-        <box size=".02 .025 .04"/>
-      </geometry>
-      <origin xyz="-0.005 ${reflect*0.01} .045"/>
-      <material name="gray"/>
-    </visual>
-    <xacro:default_inertial mass="${gripper_finger_mass}"/>
-  </link>
-  <joint name="arm_${arm}_finger_${suffix}_joint" type="revolute">
+  <joint name="arm_${arm}_finger_right_joint" type="revolute">
     <axis xyz="0 1 0"/>
     <limit effort="1000.0" lower="0.0" upper="0.548" velocity="0.5"/>
-    <origin rpy="0 0 ${reflect*pi/2-pi/2}" xyz="${reflect*0.015} 0 0"/>
+    <origin rpy="0 0 ${-reflect*pi/2-pi/2}" xyz="${-reflect*0.015} 0 0"/>
     <parent link="arm_${arm}_gripper_base"/>
-    <child link="arm_${arm}_finger_${suffix}_link"/>
-		<mimic joint="arm_${arm}_finger_${mimic}_joint" multiplier="1" offset="0"/>
+    <child link="arm_${arm}_finger_right_link"/>
+    <mimic joint="arm_${arm}_finger_left_joint" multiplier="1" offset="0"/>
   </joint>
 </xacro:macro>
@@ -80,6 +63,7 @@
     <origin rpy="0 0 0" xyz="0 0 0.05"/>
   </joint>
-  <xacro:call macro="finger" arm="${arm}" suffix="left" reflect="1"/>
-  <xacro:call macro="finger_mimic" arm="${arm}" suffix="right" mimic="left" reflect="-1"/>
+  <xacro:call macro="finger_link" arm="${arm}" suffix="left" reflect="1"/>
+  <xacro:call macro="finger_link" arm="${arm}" suffix="right" reflect="-1"/>
+  <xacro:call macro="gripper_joint" arm="${arm}" reflect="1"/>
 </xacro:macro>
 </robot>
